Commit message: Replace RGB camera for RGB-D one

File: graphslam/urdf/my_robot.xacro (robot description, xacro)
@@ -5,5 +5,5 @@
   <joint name="robot_footprint_joint" type="fixed">
     <origin xyz="0 0 0" rpy="0 0 0" />
-    <parent link="robot_footprint"/>
+    <parent link="robot_footprint" />
     <child link="chassis" />
   </joint>
@@ -11,69 +11,61 @@
     <pose>0 0 0.1 0 0 0</pose>
     <inertial>
-      <mass value="15.0"/>
-      <origin xyz="0.0 0 0" rpy=" 0 0 0"/>
-      <inertia
-          ixx="0.1" ixy="0" ixz="0"
-          iyy="0.1" iyz="0"
-          izz="0.1"
-      />
+      <mass value="15.0" />
+      <origin xyz="0.0 0 0" rpy=" 0 0 0" />
+      <inertia ixx="0.1" ixy="0" ixz="0" iyy="0.1" iyz="0" izz="0.1" />
     </inertial>
     <collision name='collision'>
-      <origin xyz="0 0 0" rpy=" 0 0 0"/>
+      <origin xyz="0 0 0" rpy=" 0 0 0" />
       <geometry>
-        <box size=".4 .2 .1"/>
+        <box size=".4 .2 .1" />
       </geometry>
     </collision>
     <visual name='chassis_visual'>
-      <origin xyz="0 0 0" rpy=" 0 0 0"/>
+      <origin xyz="0 0 0" rpy=" 0 0 0" />
       <geometry>
-        <box size=".4 .2 .1"/>
+        <box size=".4 .2 .1" />
       </geometry>
     </visual>
     <collision name='back_caster_collision'>
-      <origin xyz="-0.15 0 -0.05" rpy=" 0 0 0"/>
+      <origin xyz="-0.15 0 -0.05" rpy=" 0 0 0" />
       <geometry>
-        <sphere radius="0.0499"/>
+        <sphere radius="0.0499" />
       </geometry>
     </collision>
     <visual name='back_caster_visual'>
-      <origin xyz="-0.15 0 -0.05" rpy=" 0 0 0"/>
+      <origin xyz="-0.15 0 -0.05" rpy=" 0 0 0" />
       <geometry>
-        <sphere radius="0.05"/>
+        <sphere radius="0.05" />
       </geometry>
     </visual>
     <collision name='front_caster_collision'>
-      <origin xyz="0.15 0 -0.05" rpy=" 0 0 0"/>
+      <origin xyz="0.15 0 -0.05" rpy=" 0 0 0" />
       <geometry>
-        <sphere radius="0.0499"/>
+        <sphere radius="0.0499" />
       </geometry>
     </collision>
     <visual name='front_caster_visual'>
-      <origin xyz="0.15 0 -0.05" rpy=" 0 0 0"/>
+      <origin xyz="0.15 0 -0.05" rpy=" 0 0 0" />
       <geometry>
-        <sphere radius="0.05"/>
+        <sphere radius="0.05" />
       </geometry>
     </visual>
   </link>
   <joint type="continuous" name="left_wheel_hinge">
-    <origin xyz="0 0.15 0" rpy="0 0 0"/>
-    <child link="left_wheel"/>
-    <parent link="chassis"/>
-    <axis xyz="0 1 0" rpy="0 0 0"/>
-    <limit effort="10000" velocity="1000"/>
-    <dynamics damping="1.0" friction="1.0"/>
+    <origin xyz="0 0.15 0" rpy="0 0 0" />
+    <child link="left_wheel" />
+    <parent link="chassis" />
+    <axis xyz="0 1 0" rpy="0 0 0" />
+    <limit effort="10000" velocity="1000" />
+    <dynamics damping="1.0" friction="1.0" />
   </joint>
   <link name="left_wheel">
     <inertial>
-      <mass value="5.0"/>
-      <origin xyz="0.0 0 0" rpy="0 1.5707 1.5707"/>
-      <inertia
-          ixx="0.1" ixy="0" ixz="0"
-          iyy="0.1" iyz="0"
-          izz="0.1"
-      />
+      <mass value="5.0" />
+      <origin xyz="0.0 0 0" rpy="0 1.5707 1.5707" />
+      <inertia ixx="0.1" ixy="0" ixz="0" iyy="0.1" iyz="0" izz="0.1" />
     </inertial>
     <collision name='collision'>
-      <origin xyz="0 0 0" rpy="0 1.5707 1.5707"/>
+      <origin xyz="0 0 0" rpy="0 1.5707 1.5707" />
       <geometry>
         <cylinder radius="0.1" length="0.05" />
@@ -81,5 +73,5 @@
     </collision>
     <visual name='chassis_visual'>
-      <origin xyz="0 0 0" rpy="0 1.5707 1.5707"/>
+      <origin xyz="0 0 0" rpy="0 1.5707 1.5707" />
       <geometry>
         <cylinder radius="0.1" length="0.05" />
@@ -88,23 +80,19 @@
   </link>
   <joint type="continuous" name="right_wheel_hinge">
-    <origin xyz="0 -0.15 0" rpy="0 0 0"/>
-    <child link="right_wheel"/>
-    <parent link="chassis"/>
-    <axis xyz="0 1 0" rpy="0 0 0"/>
-    <limit effort="10000" velocity="1000"/>
-    <dynamics damping="1.0" friction="1.0"/>
+    <origin xyz="0 -0.15 0" rpy="0 0 0" />
+    <child link="right_wheel" />
+    <parent link="chassis" />
+    <axis xyz="0 1 0" rpy="0 0 0" />
+    <limit effort="10000" velocity="1000" />
+    <dynamics damping="1.0" friction="1.0" />
   </joint>
   <link name="right_wheel">
     <inertial>
-      <mass value="5.0"/>
-      <origin xyz="0.0 0 0" rpy="0 1.5707 1.5707"/>
-      <inertia
-          ixx="0.1" ixy="0" ixz="0"
-          iyy="0.1" iyz="0"
-          izz="0.1"
-      />
+      <mass value="5.0" />
+      <origin xyz="0.0 0 0" rpy="0 1.5707 1.5707" />
+      <inertia ixx="0.1" ixy="0" ixz="0" iyy="0.1" iyz="0" izz="0.1" />
     </inertial>
     <collision name='collision'>
-      <origin xyz="0 0 0" rpy="0 1.5707 1.5707"/>
+      <origin xyz="0 0 0" rpy="0 1.5707 1.5707" />
       <geometry>
         <cylinder radius="0.1" length="0.05" />
@@ -112,5 +100,5 @@
     </collision>
     <visual name='chassis_visual'>
-      <origin xyz="0 0 0" rpy="0 1.5707 1.5707"/>
+      <origin xyz="0 0 0" rpy="0 1.5707 1.5707" />
       <geometry>
         <cylinder radius="0.1" length="0.05" />
@@ -119,18 +107,14 @@
   </link>
   <joint type="fixed" name="camera_joint">
-    <origin xyz="0.2 0 0" rpy="0 0 0"/>
-    <child link="camera"/>
-    <parent link="chassis"/>
-    <axis xyz="0 1 0" rpy="0 0 0"/>
+    <origin xyz="0.2 0 0" rpy="0 0 0" />
+    <child link="camera_link" />
+    <parent link="chassis" />
+    <axis xyz="0 1 0" rpy="0 0 0" />
   </joint>
-  <link name="camera">
+  <link name="camera_link">
     <inertial>
-      <mass value="0.1"/>
-      <origin xyz="0.0 0 0" rpy="0 0 0"/>
-      <inertia
-          ixx="1e-6" ixy="0" ixz="0"
-          iyy="1e-6" iyz="0"
-          izz="1e-6"
-      />
+      <mass value="0.1" />
+      <origin xyz="0.0 0 0" rpy="0 0 0" />
+      <inertia ixx="1e-6" ixy="0" ixz="0" iyy="1e-6" iyz="0" izz="1e-6" />
     </inertial>
     <collision name='collision'>
@@ -148,18 +132,14 @@
   </link>
   <joint type="fixed" name="hokuyo_joint">
-    <origin xyz="0.15 0 0.1" rpy="0 0 0"/>
-    <child link="hokuyo"/>
-    <parent link="chassis"/>
-    <axis xyz="0 1 0" rpy="0 0 0"/>
+    <origin xyz="0.15 0 0.1" rpy="0 0 0" />
+    <child link="hokuyo" />
+    <parent link="chassis" />
+    <axis xyz="0 1 0" rpy="0 0 0" />
   </joint>
   <link name="hokuyo">
     <inertial>
-      <mass value="1e-5"/>
-      <origin xyz="0 0 0" rpy="0 0 0"/>
-      <inertia
-          ixx="1e-6" ixy="0" ixz="0"
-          iyy="1e-6" iyz="0"
-          izz="1e-6"
-      />
+      <mass value="1e-5" />
+      <origin xyz="0 0 0" rpy="0 0 0" />
+      <inertia ixx="1e-6" ixy="0" ixz="0" iyy="1e-6" iyz="0" izz="1e-6" />
     </inertial>
     <collision name='collision'>
@@ -176,3 +156,9 @@
     </visual>
   </link>
+  <joint name="camera_optical_joint" type="fixed">
+    <origin xyz="0 0 0" rpy="-1.5707 0 -1.5707" />
+    <parent link="camera_link" />
+    <child link="camera_link_optical" />
+  </joint>
+  <link name="camera_link_optical"></link>
 </robot>
